Commit message: urdf 내 파일 경로 수정

File: rby1_description/urdf/rby1.urdf (robot description, URDF)
Before this commit: robot rby1, 35 links, 34 joints
Links:
- link FT_sensor_L: geometry visual mesh filename=package://rby1_description/meshes/FT_SENSOR_L.dae
- link FT_sensor_R: geometry visual mesh filename=package://rby1_description/meshes/FT_SENSOR_R.dae
- link base: geometry visual mesh filename=package://rby1_description/meshes/base.dae
- link ee_finger_l1: geometry visual mesh filename=package://rby1_description/meshes/EE_FINGER.dae
- link ee_finger_l2: geometry visual mesh filename=package://rby1_description/meshes/EE_FINGER.dae
- link ee_finger_r1: geometry visual mesh filename=package://rby1_description/meshes/EE_FINGER.dae
- link ee_finger_r2: geometry visual mesh filename=package://rby1_description/meshes/EE_FINGER.dae
- link ee_left: geometry visual mesh filename=package://rby1_description/meshes/EE_BODY.dae
- link ee_right: geometry visual mesh filename=package://rby1_description/meshes/EE_BODY.dae
- link link_head_0: geometry visual mesh filename=package://rby1_description/meshes/PAN_TILT_1.dae
- link link_head_1: geometry visual mesh filename=package://rby1_description/meshes/PAN_TILT_2.dae
- link link_head_2: geometry visual mesh filename=package://rby1_description/meshes/PAN_TILT_3.dae
- link link_left_arm_0: geometry collision sphere radius=0.075; visual mesh filename=package://rby1_description/meshes/LINK_14.dae
- link link_left_arm_1: geometry collision sphere radius=0.050; visual mesh filename=package://rby1_description/meshes/LINK_15.dae
- link link_left_arm_2: geometry collision sphere radius=0.05; visual mesh filename=package://rby1_description/meshes/LINK_16.dae
- link link_left_arm_3: geometry collision sphere radius=0.04; visual mesh filename=package://rby1_description/meshes/LINK_17.dae
- link link_left_arm_4: geometry collision sphere radius=0.035; visual mesh filename=package://rby1_description/meshes/LINK_18.dae
- link link_left_arm_5: geometry collision sphere radius=0.075; visual mesh filename=package://rby1_description/meshes/LINK_19.dae
- link link_left_arm_6: geometry visual mesh filename=package://rby1_description/meshes/LINK_20.dae
- link link_right_arm_0: geometry collision sphere radius=0.075; visual mesh filename=package://rby1_description/meshes/LINK_7.dae
- link link_right_arm_1: geometry collision sphere radius=0.05; visual mesh filename=package://rby1_description/meshes/LINK_8.dae
- link link_right_arm_2: geometry collision sphere radius=0.05; visual mesh filename=package://rby1_description/meshes/LINK_9.dae
- link link_right_arm_3: geometry collision sphere radius=0.04; visual mesh filename=package://rby1_description/meshes/LINK_10.dae
- link link_right_arm_4: geometry collision sphere radius=0.035; visual mesh filename=package://rby1_description/meshes/LINK_11.dae
- link link_right_arm_5: geometry collision sphere radius=0.075; visual mesh filename=package://rby1_description/meshes/LINK_12.dae
- link link_right_arm_6: geometry visual mesh filename=package://rby1_description/meshes/LINK_13.dae
- link link_torso_0: geometry collision sphere radius=0.105; visual mesh filename=package://rby1_description/meshes/LINK_1.dae
- link link_torso_1: geometry collision sphere radius=0.115; visual mesh filename=package://rby1_description/meshes/LINK_2.dae
- link link_torso_2: geometry collision sphere radius=0.095; visual mesh filename=package://rby1_description/meshes/LINK_3.dae
- link link_torso_3: geometry visual mesh filename=package://rby1_description/meshes/LINK_4.dae
- link link_torso_4: geometry collision sphere radius=0.105; visual mesh filename=package://rby1_description/meshes/LINK_5.dae
- link link_torso_5: geometry collision sphere radius=0.155; visual mesh filename=package://rby1_description/meshes/LINK_6.dae
- link wheel_l: geometry visual mesh filename=package://rby1_description/meshes/WHEEL.dae
- link wheel_r: geometry visual mesh filename=package://rby1_description/meshes/WHEEL.dae
